File: sensorPlatform/schematic1.brd (EAGLE design)
At the start: 100 x 80 mm, 3 parts

Commit message: Add files via upload
Parts:
- moved B1 100.3 mm to (82.5, 24.1)
- moved MS1 66.6 mm to (15.2, 5.08)
- moved U$1 45.8 mm to (-74.9, 43.2)
Connections:
- removed net VCC: B1.21, MS1.2
- new net 3.3V: MS1.4, U$1.15
- new net 3V: B1.21
- new net VBAT: MS1.28
- net GND: no longer MS1.4
Changed lines of the file:
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@@
 <?xml version="1.0" encoding="utf-8"?>
 <!DOCTYPE eagle SYSTEM "eagle.dtd">
-<eagle version="8.6.0">
+<eagle version="8.6.2">
 <drawing>
 <settings>
@@
 <layers>
 <layer number="1" name="Top" color="4" fill="1" visible="yes" active="yes"/>
+<layer number="2" name="Route2" color="1" fill="3" visible="no" active="yes"/>
+<layer number="3" name="Route3" color="4" fill="3" visible="no" active="yes"/>
+<layer number="4" name="Route4" color="1" fill="4" visible="no" active="yes"/>
+<layer number="5" name="Route5" color="4" fill="4" visible="no" active="yes"/>
+<layer number="6" name="Route6" color="1" fill="8" visible="no" active="yes"/>
+<layer number="7" name="Route7" color="4" fill="8" visible="no" active="yes"/>
+<layer number="8" name="Route8" color="1" fill="2" visible="no" active="yes"/>
+<layer number="9" name="Route9" color="4" fill="2" visible="no" active="yes"/>
+<layer number="10" name="Route10" color="1" fill="7" visible="no" active="yes"/>
+<layer number="11" name="Route11" color="4" fill="7" visible="no" active="yes"/>
+<layer number="12" name="Route12" color="1" fill="5" visible="no" active="yes"/>
+<layer number="13" name="Route13" color="4" fill="5" visible="no" active="yes"/>
+<layer number="14" name="Route14" color="1" fill="6" visible="no" active="yes"/>
+<layer number="15" name="Route15" color="4" fill="6" visible="no" active="yes"/>
 <layer number="16" name="Bottom" color="1" fill="1" visible="yes" active="yes"/>
 <layer number="17" name="Pads" color="2" fill="1" visible="yes" active="yes"/>
@@
 </autorouter>
 <elements>
-<element name="B1" library="SparkFun-Boards" library_urn="urn:adsk.eagle:library:509" package="SPARKFUN_PRO_MICRO" package3d_urn="urn:adsk.eagle:package:37326/1" value="SPARKFUN_PRO_MICRO" x="-17.78" y="25.4"/>
-<element name="U$1" library="adafruit" library_urn="urn:adsk.eagle:library:420" package="TQFP44" value="ATMEGA32U4-AU" x="-43.18" y="10.16"/>
-<element name="MS1" library="adafruit" library_urn="urn:adsk.eagle:library:420" package="FEATHERWING" value="FEATHERWING" x="-34.29" y="-39.37"/>
+<element name="B1" library="SparkFun-Boards" library_urn="urn:adsk.eagle:library:509" package="SPARKFUN_PRO_MICRO" package3d_urn="urn:adsk.eagle:package:37326/1" value="SPARKFUN_PRO_MICRO" x="82.55" y="24.13"/>
+<element name="U$1" library="adafruit" library_urn="urn:adsk.eagle:library:420" package="TQFP44" value="ATMEGA32U4-AU" x="-74.93" y="43.18"/>
+<element name="MS1" library="adafruit" library_urn="urn:adsk.eagle:library:420" package="FEATHERWING" value="FEATHERWING" x="15.24" y="5.08"/>
 </elements>
 <signals>
@@
 <contactref element="B1" pad="23"/>
 <contactref element="B1" pad="3"/>
-<contactref element="MS1" pad="4"/>
-<wire x1="-25.4" y1="30.48" x2="-20.32" y2="-38.1" width="0" layer="19" extent="1-1"/>
-<wire x1="-25.4" y1="33.02" x2="-25.4" y2="30.48" width="0" layer="19" extent="1-1"/>
-<wire x1="-10.16" y1="35.56" x2="-25.4" y2="33.02" width="0" layer="19" extent="1-1"/>
+<wire x1="74.93" y1="31.75" x2="90.17" y2="34.29" width="0" layer="19" extent="1-1"/>
+<wire x1="74.93" y1="29.21" x2="74.93" y2="31.75" width="0" layer="19" extent="1-1"/>
 </signal>
 <signal name="RAW">
 <contactref element="B1" pad="24"/>
 </signal>
-<signal name="VCC">
-<contactref element="MS1" pad="2"/>
+<signal name="3V">
 <contactref element="B1" pad="21"/>
-<wire x1="-10.16" y1="30.48" x2="-25.4" y2="-38.1" width="0" layer="19" extent="1-1"/>
+</signal>
+<signal name="3.3V">
+<contactref element="MS1" pad="4"/>
+<contactref element="U$1" pad="15"/>
+<wire x1="29.21" y1="6.35" x2="-76.53" y2="37.38" width="0" layer="19" extent="1-1"/>
+</signal>
+<signal name="VBAT">
+<contactref element="MS1" pad="28"/>
 </signal>
 </signals>
