File: charging_and_sensors/lt3652_charger.sch (EAGLE design)
At the start: 20 parts, among them U1 LT3652

Commit message: Add files via upload
Parts:
- removed D8: (no value), adafruit:DIODEDO-1N4148
- added B=3380: THERMISTOR-5, varistor:THERMISTOR-5
- added BAT2: 3.7, special:BATTERY
- added LED1, LED2, LED3, LED4: (no value), adafruit:LED5MM
- added R10: 223k, adafruit:R-US_0204/2V
- added R9: 10k, adafruit:R-US_0204/2V
- BAT1: value (none) -> 3.7V
- C1: value (none) -> .68µF
- C2: value (none) -> 10µF
- C4: value (none) -> 1µF
- L1: value (none) -> 5µH
- R1: value (none) -> 7k
- R2: value (none) -> 9k
- R3: value (none) -> 10k
- R4: value (none) -> 80k
- R5: value (none) -> 20k
- R6: value (none) -> 30k
- R7: value (none) -> 330k
- R8: value (none) -> .1
Connections:
- new net N$12: R9.1, U1.!CHRG
- new net N$13: B=3380.2, U1.NTC
- new net N$4: LED1.C, LED2.A, R3.2
- net 0: now also B=3380.1, BAT2.-
- net LOAD: now also LED1.A, LED2.C, LED3.A, LED4.C; no longer D8.A
- net N$5: now also LED3.C, LED4.A; no longer D8.C, R3.2
- net N$8: now also BAT2.+
- net N$9: no longer U1.VFB
Other:
- note removed: "Also, this chip and the other chip do go through the necessary preconditioning phase, constant current phase, and constant voltage phase"
- note removed: "Concerns: Batteries in series would result in voltage of 7.4, higher than 6V output of solar panel. In parallel, current splits between two packs so they would charge in half the time? Not certain if this chip can support 6-cell charging like other chip. It's not specified. On the plus side, this uses charging cycles on a clock timer instead of temperature monitoring. Both are MPPT."
- moved on the sheet: C2, R3
